Commit message: add lec3 exercise

File: catkin_ws/src/autolabor_description/urdf/autolabor_mini.urdf (robot description, URDF)
Before this commit: robot autolabor_description, 1 links, 0 joints
Links:
- added link lidar
Joints:
- added joint joint0: type fixed, parent base_link, child lidar, origin xyz=0. 0. 0.15
